Commit message: ros2 control

File: xarm_description/xarmbot/urdf/xarm.urdf (robot description, URDF)
Before this commit: robot xarm, 6 links, 6 joints
Links:
- removed link xarm_base_link
- added link base_link; collision mesh filename=package://xarm_description/xarmbot/meshes/stls/base.stl scale=1.0 1.0 1.0; visual mesh filename=package://xarm_description/xarmbot/meshes/stls/base.stl scale=1.0 1.0 1.0
- link xarm_7_link: geometry collision mesh filename=package://ros2_control_demo_description/xarmbot/meshes/stls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 scale=1.0 1.0 1.0; visual mesh filename=package://ros2_control_demo_description/xarmbot/meshes/stls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 scale=1.0 1.0 1.0
Joints:
- joint xarm_6_joint: parent xarm_base_link -> base_link

File: xarm_description/xarmbot/urdf/xarm_world.urdf.xacro (robot description, xacro)
@@ -2,10 +2,10 @@
 <robot xmlns:xacro="http://ros.org/wiki/xacro" name="xarm">
     <xacro:property name="eef" value="eef_3_finger"/>
-    <xacro:include filename="$(find ros2_control_demo_description)/xarmbot/urdf/xarm.urdf"/>
+    <xacro:include filename="$(find xarm_description)/xarmbot/urdf/xarm.urdf"/>
     <link name="world"/>
     <xacro:arg name="initial_z" default="0.0"/>
     <joint name="world_joint" type="fixed">
         <parent link="world"/>
-        <child link="xarm_base_link"/>
+        <child link="base_link"/>
         <origin xyz="0.0 0.0 $(arg initial_z)" rpy="0.0 0.0 0.0"/>
     </joint>

Commit message: update description

File: xarm_description/xarmbot/urdf/xarm.urdf (robot description, URDF)
Before this commit: robot xarm, 6 links, 6 joints
Links:
- removed link xarm_7_link
Joints:
- removed joint xarm_7_joint
- joint xarm_3_joint: origin xyz=0 0.0 0.030 rpy=0 0 0 -> xyz=0 0.0 0.093 rpy=0 0 0; parent xarm_7_link -> xarm_4_link

File: xarm_description/xarmbot/urdf/xarm_world.urdf.xacro (robot description, xacro)
@@ -1,5 +1,5 @@
 <?xml version="1.0"?>
 <robot xmlns:xacro="http://ros.org/wiki/xacro" name="xarm">
-    <xacro:property name="eef" value="eef_3_finger"/>
+    <xacro:property name="eef" value="eef_2_finger"/>
     <xacro:include filename="$(find xarm_description)/xarmbot/urdf/xarm.urdf"/>
     <link name="world"/>
